File: MainPCB.kicad_sch (KiCad schematic)
At the start: 59 parts, among them J1 RaspberryPi, J10 Conn_01x02, J2 Conn_01x05, J3 Screw_Terminal_01x02, J4 Conn_01x02, J5 Conn_01x06, J6 Conn_01x03_Pin, J7 Conn_01x05, J8 Conn_01x12, J9 Conn_01x02, M1 Motor_DC, M2 Motor_DC, M3 Motor_DC, M4 Motor_DC, M5 Motor_DC, SW1 SW_SPDT, SW2 SW_SPDT, SW3 SW_SPDT, SW4 SW_SPDT, U1 Teensy4.1, U10 Compass, U11 V_Regulator5v, U12 RockerSwitch, U13 V_Regulator3.3v, U2 VNH Driver, U3 VNH Driver, U4 VNH Driver, U5 VNH Driver, U6 TSOP25xx, U7 V_Regulator5v, U8 VNH Driver

Commit message: Finished Routing
Parts:
- removed C11, C12: .1uf, Capacitor_SMD:C_0805_2012Metric, symbol Device:C
- C1: value 10uf -> .1uf
- C6, C8, C9: value .1uf -> 10uf
Connections:
- net 5V: no longer J8.9 (Pin_9)

Commit message: fixed ultrasonic voltages
Connections:
- net 3.3V: no longer J2.1 (Pin_1), J7.1 (Pin_1)
- net 5V: now also J2.1 (Pin_1), J7.1 (Pin_1)
Changed lines of the file:
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@@
 	)
 	(junction
-		(at 302.26 218.44)
-		(diameter 0)
-		(color 0 0 0 0)
-	)
-	(junction
 		(at 88.9 44.45)
 		(diameter 0)
@@
 	(wire
 		(pts
-			(xy 302.26 218.44) (xy 302.26 237.49)
-		)
-		(stroke
-			(width 0)
-			(type default)
-		)
-	)
-	(wire
-		(pts
 			(xy 100.33 168.91) (xy 86.36 168.91)
 		)
@@
 	(wire
 		(pts
-			(xy 297.18 218.44) (xy 302.26 218.44)
-		)
-		(stroke
-			(width 0)
-			(type default)
-		)
-	)
-	(wire
-		(pts
 			(xy 100.33 119.38) (xy 100.33 124.46)
 		)
@@
 	(wire
 		(pts
-			(xy 302.26 207.01) (xy 302.26 218.44)
+			(xy 302.26 207.01) (xy 302.26 237.49)
 		)
 		(stroke
@@
 	(rectangle
 		(start 316.23 119.38)
-		(end 386.08 166.37)
+		(end 371.475 159.385)
 		(stroke
 			(width 0)
@@
 		)
 	)
+	(global_label "5V"
+		(shape input)
+		(at 302.26 220.98 180)
+		(fields_autoplaced yes)
+		(effects
+			(font
+				(size 1.27 1.27)
+			)
+			(justify right)
+		)
+		(property "Intersheetrefs" "${INTERSHEET_REFS}"
+			(at 296.9767 220.98 0)
+			(effects
+				(font
+					(size 1.27 1.27)
+				)
+				(justify right)
+				(hide yes)
+			)
+		)
+	)
 	(global_label "DIR1B"
 		(shape input)
@@
 			(effects
 				(font
-					(size 1.27 1.27)
-				)
-				(justify right)
-				(hide yes)
-			)
-		)
-	)
-	(global_label "3.3V"
-		(shape input)
-		(at 297.18 218.44 180)
-		(fields_autoplaced yes)
-		(effects
-			(font
-				(size 1.27 1.27)
-			)
-			(justify right)
-		)
-		(property "Intersheetrefs" "${INTERSHEET_REFS}"
-			(at 290.0824 218.44 0)
-			(effects
-				(font
